Commit message: Starting work on assignment6.

File: body.urdf (robot description, URDF)
Before this commit: robot robot, 3 links, 2 joints
Links:
- removed link BackLeg
- removed link FrontLeg
- removed link Torso
- added link Segment0, mass 1; collision box size=1 1 1; visual box size=1 1 1
- added link Segment1, mass 1; collision box size=1.0924953723456063 1.015645875740245 0.9814292846517929; visual box size=1.0924953723456063 1.015645875740245 0.9814292846517929
- added link Segment2, mass 1; collision box size=1.080045409976834 1.0692359101377207 1.1311582935249191; visual box size=1.080045409976834 1.0692359101377207 1.1311582935249191
- added link Segment3, mass 1; collision box size=0.9470133113132242 0.8235215383790513 0.8089023135879772; visual box size=0.9470133113132242 0.8235215383790513 0.8089023135879772
- added link Segment4, mass 1; collision box size=1.1265562648381051 1.17798275159962 1.0908279034967356; visual box size=1.1265562648381051 1.17798275159962 1.0908279034967356
- added link Segment5, mass 1; collision box size=0.9834571929534583 0.8254602922912071 1.1218257947700108; visual box size=0.9834571929534583 0.8254602922912071 1.1218257947700108
Joints:
- removed joint Torso_BackLeg
- removed joint Torso_FrontLeg
- added joint Segment0_Segment1: type revolute, parent Segment0, child Segment1, origin xyz=0.5 0 0.5 rpy=0 0 0, axis -0.4838180274140158 -0.5587355338016065 0.9671818654895519, limit lower=-3.14159 upper=3.14159 effort=0.0 velocity=0.0
- added joint Segment1_Segment2: type revolute, parent Segment1, child Segment2, origin xyz=1.0924953723456063 0 0.5 rpy=0 0 0, axis -0.06893311404062263 -0.9841789111290216 -0.6736050038555617, limit lower=-3.14159 upper=3.14159 effort=0.0 velocity=0.0
- added joint Segment2_Segment3: type revolute, parent Segment2, child Segment3, origin xyz=1.080045409976834 0 0.5 rpy=0 0 0, axis -0.15858214011468896 -0.11166173757064746 -0.26331830937753997, limit lower=-3.14159 upper=3.14159 effort=0.0 velocity=0.0
- added joint Segment3_Segment4: type revolute, parent Segment3, child Segment4, origin xyz=0.9470133113132242 0 0.5 rpy=0 0 0, axis -0.8361628367649234 -0.010111355696310387 -0.010394728950527732, limit lower=-3.14159 upper=3.14159 effort=0.0 velocity=0.0
- added joint Segment4_Segment5: type revolute, parent Segment4, child Segment5, origin xyz=1.1265562648381051 0 0.5 rpy=0 0 0, axis -0.5827953822025236 -0.028290603313307683 0.2249244376279409, limit lower=-3.14159 upper=3.14159 effort=0.0 velocity=0.0

Commit message: Starting work on 3d_creature.

File: body.urdf (robot description, URDF)
Before this commit: robot robot, 6 links, 5 joints
Links:
- removed link Segment0
- removed link Segment1
- removed link Segment2
- removed link Segment3
- removed link Segment4
- removed link Segment5
- added link Leg0Part0, mass 1; collision box size=1.1030113152030687 0.9754179224671128 0.8604722786232286; visual box size=1.1030113152030687 0.9754179224671128 0.8604722786232286
- added link Leg0Part1, mass 1; collision box size=0.8656453219854529 1.1029983078268184 1.197933512023124; visual box size=0.8656453219854529 1.1029983078268184 1.197933512023124
- added link Leg0Part2, mass 1; collision box size=0.933899927977874 0.92075873666361 1.143524871256302; visual box size=0.933899927977874 0.92075873666361 1.143524871256302
- added link Leg0Part3, mass 1; collision box size=1.1803092722411916 0.8869800766287163 0.8142870154775035; visual box size=1.1803092722411916 0.8869800766287163 0.8142870154775035
- added link Leg1Part0, mass 1; collision box size=0.8753017405951553 0.956200697220923 1.0929183718340787; visual box size=0.8753017405951553 0.956200697220923 1.0929183718340787
- added link Leg1Part1, mass 1; collision box size=0.8883158315290192 0.8313430949062591 1.1170015288570119; visual box size=0.8883158315290192 0.8313430949062591 1.1170015288570119
- added link Leg1Part2, mass 1; collision box size=0.8659120026039243 0.9660261090967304 0.9404222437012564; visual box size=0.8659120026039243 0.9660261090967304 0.9404222437012564
- added link Leg2Part0, mass 1; collision box size=0.8980621009668063 1.1172809548833915 0.9943571090904945; visual box size=0.8980621009668063 1.1172809548833915 0.9943571090904945
- added link Leg2Part1, mass 1; collision box size=0.8796697392683405 1.0319023935346734 0.9036954501562088; visual box size=0.8796697392683405 1.0319023935346734 0.9036954501562088
- added link Leg2Part2, mass 1; collision box size=1.1316236480826074 0.8881731638026933 0.9728294013273598; visual box size=1.1316236480826074 0.8881731638026933 0.9728294013273598
- added link Torso0, mass 1; collision box size=1 1 1; visual box size=1 1 1
- added link Torso1, mass 1; collision box size=0.9695537026518543 0.9296039444427876 1.0621668216823428; visual box size=0.9695537026518543 0.9296039444427876 1.0621668216823428
- added link Torso2, mass 1; collision box size=0.9035973902234821 1.1760523936488256 0.8308698651812529; visual box size=0.9035973902234821 1.1760523936488256 0.8308698651812529
- added link Torso3, mass 1; collision box size=1.197673103203757 0.9635995334177174 0.9247766475615576; visual box size=1.197673103203757 0.9635995334177174 0.9247766475615576
- added link Torso4, mass 1; collision box size=0.9603685175485326 0.9085393608144646 1.086767863499313; visual box size=0.9603685175485326 0.9085393608144646 1.086767863499313
- added link Torso5, mass 1; collision box size=0.9718608551972029 0.8202076078114079 1.0910644796185491; visual box size=0.9718608551972029 0.8202076078114079 1.0910644796185491
- added link Torso6, mass 1; collision box size=0.9526681064094709 0.9556132562839474 0.9975177249842662; visual box size=0.9526681064094709 0.9556132562839474 0.9975177249842662
- added link Torso7, mass 1; collision box size=0.9414343349818113 0.891754380619203 0.8652890132089937; visual box size=0.9414343349818113 0.891754380619203 0.8652890132089937
Joints:
- removed joint Segment0_Segment1
- removed joint Segment1_Segment2
- removed joint Segment2_Segment3
- removed joint Segment3_Segment4
- removed joint Segment4_Segment5
- added joint Leg0Part0_Leg0Part1: type revolute, parent Leg0Part0, child Leg0Part1, origin xyz=0.5988365516018785 0.9635995334177174 1 rpy=0 0 0, axis 0.09608431632267922 0.25371891269312896 -0.6827770249468936, limit lower=-3.14159 upper=3.14159 effort=0.0 velocity=0.0
- added joint Leg0Part1_Leg0Part2: type revolute, parent Leg0Part1, child Leg0Part2, origin xyz=0.5988365516018785 1.1029983078268184 1 rpy=0 0 0, axis 0.6452270713803427 0.18412452364335552 0.5755138571126377, limit lower=-3.14159 upper=3.14159 effort=0.0 velocity=0.0
- added joint Leg0Part2_Leg0Part3: type revolute, parent Leg0Part2, child Leg0Part3, origin xyz=0.5988365516018785 0.92075873666361 1 rpy=0 0 0, axis -0.1779721827932379 0.5400663100503569 -0.7058654627298888, limit lower=-3.14159 upper=3.14159 effort=0.0 velocity=0.0
- added joint Leg1Part0_Leg1Part1: type revolute, parent Leg1Part0, child Leg1Part1, origin xyz=0.48593042759860144 0.8202076078114079 1 rpy=0 0 0, axis 0.9282242309141358 0.10752231085100661 0.5801033156760949, limit lower=-3.14159 upper=3.14159 effort=0.0 velocity=0.0
- added joint Leg1Part1_Leg1Part2: type revolute, parent Leg1Part1, child Leg1Part2, origin xyz=0.48593042759860144 0.8313430949062591 1 rpy=0 0 0, axis 0.9016084124785304 0.2763693928557571 0.2338327536826219, limit lower=-3.14159 upper=3.14159 effort=0.0 velocity=0.0
- added joint Leg2Part0_Leg2Part1: type revolute, parent Leg2Part0, child Leg2Part1, origin xyz=0.47071716749090564 0 0.8652890132089937 rpy=0 0 0, axis 0.5452140259437639 0.40143222775325804 -0.7159613710023791, limit lower=-3.14159 upper=3.14159 effort=0.0 velocity=0.0
- added joint Leg2Part1_Leg2Part2: type revolute, parent Leg2Part1, child Leg2Part2, origin xyz=0.47071716749090564 0 0.9036954501562088 rpy=0 0 0, axis 0.11853143890907702 -0.9133026410125127 -0.4552085564551127, limit lower=-3.14159 upper=3.14159 effort=0.0 velocity=0.0
- added joint Torso0_Torso1: type revolute, parent Torso0, child Torso1, origin xyz=0.5 0 0.5 rpy=0 0 0, axis -0.3620422953719551 -0.1076388175376588 -0.48399222470844094, limit lower=-3.14159 upper=3.14159 effort=0.0 velocity=0.0
- added joint Torso1_Torso2: type revolute, parent Torso1, child Torso2, origin xyz=0.9695537026518543 0 0.5 rpy=0 0 0, axis 0.2632852340825864 -0.41738356722986336 -0.7102851796135334, limit lower=-3.14159 upper=3.14159 effort=0.0 velocity=0.0
- added joint Torso2_Leg0Part0: type revolute, parent Torso2, child Leg0Part0, origin xyz=0.5988365516018785 0.4817997667088587 1 rpy=0 0 0, axis 0.5893118437479956 -0.08297866954598865 -0.08135778728074983, limit lower=-3.14159 upper=3.14159 effort=0.0 velocity=0.0
- added joint Torso2_Torso3: type revolute, parent Torso2, child Torso3, origin xyz=0.9035973902234821 0 0.5 rpy=0 0 0, axis 0.07320656989593566 -0.12372180153913503 0.3169935347172319, limit lower=-3.14159 upper=3.14159 effort=0.0 velocity=0.0
- added joint Torso3_Torso4: type revolute, parent Torso3, child Torso4, origin xyz=1.197673103203757 0 0.5 rpy=0 0 0, axis 0.05361659702012811 0.7177841702778069 -0.18849657222719185, limit lower=-3.14159 upper=3.14159 effort=0.0 velocity=0.0
- added joint Torso4_Leg1Part0: type revolute, parent Torso4, child Leg1Part0, origin xyz=0.48593042759860144 0.41010380390570395 1 rpy=0 0 0, axis 0.9252580063354496 -0.9457009334554969 -0.8673855203410061, limit lower=-3.14159 upper=3.14159 effort=0.0 velocity=0.0
- added joint Torso4_Torso5: type revolute, parent Torso4, child Torso5, origin xyz=0.9603685175485326 0 0.5 rpy=0 0 0, axis -0.19933438068376796 -0.8555924102337855 -0.49813784565631236, limit lower=-3.14159 upper=3.14159 effort=0.0 velocity=0.0
- added joint Torso5_Torso6: type revolute, parent Torso5, child Torso6, origin xyz=0.9718608551972029 0 0.5 rpy=0 0 0, axis 0.2632343226361771 0.731630118745048 0.6622066634075487, limit lower=-3.14159 upper=3.14159 effort=0.0 velocity=0.0
- added joint Torso6_Leg2Part0: type revolute, parent Torso6, child Leg2Part0, origin xyz=0.47071716749090564 0 1.4326445066044968 rpy=0 0 0, axis -0.9249423655112667 -0.13039525230431548 -0.7582970966684726, limit lower=-3.14159 upper=3.14159 effort=0.0 velocity=0.0
- added joint Torso6_Torso7: type revolute, parent Torso6, child Torso7, origin xyz=0.9526681064094709 0 0.5 rpy=0 0 0, axis -0.4342435775440774 0.06615945872923823 0.7630212421054823, limit lower=-3.14159 upper=3.14159 effort=0.0 velocity=0.0
